File: hardware/main.brd (EAGLE design)
At the start: 64.8 x 34 mm, 10 parts, among them U1 TXB0101_DBV_6, U2 SST25VF080BS2AF

Commit message: Connected pullup resistor on USB
Connections:
- removed net UBSMON: R1.2
- net USBMON: now also R1.2
Routing:
- net USBMON: track 0.00 -> 23.2 mm
Changed lines of the file:
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@@
 <signal name="USBMON">
 <contactref element="U1" pad="3"/>
-</signal>
-<signal name="UBSMON">
 <contactref element="R1" pad="2"/>
+<wire x1="53.975" y1="14.975" x2="53.71" y2="15.24" width="0.254" layer="1"/>
+<wire x1="53.71" y1="15.24" x2="52.705" y2="15.24" width="0.254" layer="1"/>
+<wire x1="52.705" y1="15.24" x2="52.705" y2="19.685" width="0.254" layer="1"/>
+<wire x1="52.705" y1="19.685" x2="52.07" y2="20.32" width="0.254" layer="1"/>
+<wire x1="52.07" y1="20.32" x2="40.005" y2="20.32" width="0.254" layer="1"/>
+<wire x1="40.005" y1="20.32" x2="39.29" y2="21.035" width="0.254" layer="1"/>
+<wire x1="39.29" y1="21.035" x2="39.29" y2="24.45" width="0.254" layer="1"/>
 </signal>
 <signal name="ENEXT">
