File: main.brd (EAGLE design)
At the start: 64.8 x 34 mm, 7 parts, among them U1 LM3940SOT223

Commit message: Finalized documentation and added open source licensing and logos
Parts:
- added U$1: (no value), SparkFun-Aesthetics:OSHW-LOGO-S
Changed lines of the file:
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@@
 <attribute name="VALUE" x="31.115" y="7.62" size="1.27" layer="27" rot="R90"/>
 </element>
+<element name="U$1" library="SparkFun-Aesthetics" package="OSHW-LOGO-S" value="" x="35.56" y="22.86"/>
 </elements>
 <signals>
